File: WifiTracker/WifiTracker.brd (EAGLE design)
At the start: 78.7 x 50.5 mm, 27 parts, among them Y1 16MHz

Commit message: Updated Boards, mainly changing up the Servomotor print due to cluttering
Changed lines of the file:
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@@
 <?xml version="1.0" encoding="utf-8"?>
 <!DOCTYPE eagle SYSTEM "eagle.dtd">
-<eagle version="9.3.2">
+<eagle version="9.1.3">
 <drawing>
 <settings>
@@
 </element>
 <element name="R6" library="eagle-ltspice" library_urn="urn:adsk.eagle:library:217" package="R1210" package3d_urn="urn:adsk.eagle:package:13299/1" value="10kΩ" x="95.377" y="24.13" smashed="yes" rot="MR180">
-<attribute name="NAME" x="95.377" y="20.955" size="1.27" layer="26" rot="MR180"/>
+<attribute name="NAME" x="97.917" y="24.765" size="1.27" layer="26" rot="MR180"/>
 <attribute name="SPICEMODEL" value="NONE" x="95.377" y="24.13" size="1.778" layer="28" rot="MR180" display="off"/>
 <attribute name="SPICEPREFIX" value="R" x="95.377" y="24.13" size="1.778" layer="28" rot="MR180" display="off"/>
-<attribute name="VALUE" x="92.837" y="27.305" size="1.27" layer="28" rot="MR180"/>
+<attribute name="VALUE" x="94.107" y="22.225" size="1.27" layer="28" rot="MR180"/>
 </element>
 <element name="R1" library="eagle-ltspice" library_urn="urn:adsk.eagle:library:217" package="R1210" package3d_urn="urn:adsk.eagle:package:13299/1" value="10KΩ" x="52.07" y="58.42" smashed="yes" rot="MR180">
@@
 <wire x1="50.67" y1="54.61" x2="50.8" y2="54.48" width="0.8128" layer="16"/>
 <wire x1="50.8" y1="54.48" x2="50.8" y2="52.07" width="0.8128" layer="16"/>
-<wire x1="50.8" y1="52.07" x2="50.815" y2="52.085" width="0.8128" layer="16"/>
-<wire x1="50.815" y1="52.085" x2="56.5925" y2="52.085" width="0.8128" layer="16"/>
+<wire x1="50.8" y1="52.07" x2="56.5775" y2="52.07" width="0.8128" layer="16"/>
+<wire x1="56.5775" y1="52.07" x2="56.5925" y2="52.085" width="0.8128" layer="16"/>
 </signal>
 <signal name="5VCC" class="1">
