File: WifiTracker2/WifiTracker.sch (EAGLE design)
At the start: 27 parts, among them Y1 16MHz

Commit message: update
Connections:
- net 3VCC: no longer 3V_REG.OUT_(TAB)
Changed lines of the file:
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@@
 <pinref part="3V_REG" gate="G$1" pin="OUT"/>
 <junction x="304.8" y="-25.4"/>
-<pinref part="3V_REG" gate="G$1" pin="OUT_(TAB)"/>
-<wire x1="304.8" y1="-27.94" x2="304.8" y2="-25.4" width="0.1524" layer="91"/>
 </segment>
 <segment>
